Commit message: Calibrate bottom camera for 1.1

File: robots/drone_1.1.urdf.xacro (robot description, xacro)
@@ -50,5 +50,5 @@
         <parent link="quad" />
         <child link="bottom_camera_link" />
-        <origin xyz="0 0 -0.04" rpy="0 ${pi/2} ${-pi/2}" />
+        <origin xyz="0 0 -0.04" rpy="0 ${pi/2} 0" />
     </joint>
     <xacro:property name="side_camera_x" value="0.0898" />
