Commit message: added v1.5

File: robots/drone_1.5.urdf.xacro (robot description, xacro)
@@ -9,5 +9,7 @@
     <link name="foot3" />
     <link name="foot4" />
+    <!--
     <link name="bottom_camera_link" />
+    -->
     <joint name="quad_to_center_of_lift" type="fixed">
         <parent link="quad" />
@@ -18,5 +20,5 @@
         <parent link="quad" />
         <child link="lidarlite" />
-        <origin xyz="-0.107 0 0.015" rpy="0 ${pi/2} 0" />
+        <origin xyz="-0.115 0 0.055" rpy="0 ${pi/2} 0" />
     </joint>
     <joint name="quad_to_base_footprint" type="fixed">
@@ -37,4 +39,5 @@
     <xacro:foot name="foot3" reflect_x="-1" reflect_y="-1" />
     <xacro:foot name="foot4" reflect_x="1" reflect_y="-1" />
+    <!--
     <joint name="quad_to_bottom_camera_link" type="fixed">
         <parent link="quad" />
@@ -42,3 +45,4 @@
         <origin xyz="0 0 0" rpy="0 ${pi/2} 0" />
     </joint>
+    -->
 </robot>

Commit message: filled out urdf files

File: robots/drone_1.5.urdf.xacro (robot description, xacro)
@@ -4,4 +4,5 @@
     <link name="center_of_lift" />
     <link name="lidarlite" />
+    <link name="short_distance_lidar" />
     <link name="base_footprint" />
     <link name="foot1" />
@@ -20,10 +21,15 @@
         <parent link="quad" />
         <child link="lidarlite" />
-        <origin xyz="-0.115 0 0.055" rpy="0 ${pi/2} 0" />
+        <origin xyz="-0.115 0 -0.032" rpy="0 ${pi/2} 0" />
+    </joint>
+ <joint name="quad_to_short_distance_lidar" type="fixed">
+        <parent link="quad" />
+        <child link="short_distance_lidar" />
+        <origin xyz="0.08 -0.032 -0.035" rpy="0 ${pi/2} 0" />
     </joint>
     <joint name="quad_to_base_footprint" type="fixed">
         <parent link="quad" />
         <child link="base_footprint" />
-        <origin xyz="0 0 -0.06" />
+        <origin xyz="0 0 -0.07" />
     </joint>
     <xacro:property name="foot_dist" value="0.1415" />

Commit message: Change from lidarlite to tfmini

File: robots/drone_1.5.urdf.xacro (robot description, xacro)
@@ -18,7 +18,7 @@
         <origin xyz="0 0 0.065" />
     </joint>
-    <joint name="quad_to_lidarlite" type="fixed">
+    <joint name="quad_to_tfmini" type="fixed">
         <parent link="quad" />
-        <child link="lidarlite" />
+        <child link="tfmini" />
         <origin xyz="-0.115 0 -0.032" rpy="0 ${pi/2} 0" />
     </joint>

Commit message: Fix 1.5 urdf

File: robots/drone_1.5.urdf.xacro (robot description, xacro)
@@ -1,7 +1,7 @@
 <?xml version="1.0"?>
-<robot xmlns:xacro="http://www.ros.org/wiki/xacro" name="天雷">
+<robot xmlns:xacro="http://www.ros.org/wiki/xacro" name="greased_lightning">
     <link name="quad" />
     <link name="center_of_lift" />
-    <link name="lidarlite" />
+    <link name="tfmini" />
     <link name="short_distance_lidar" />
     <link name="base_footprint" />
@@ -23,5 +23,5 @@
         <origin xyz="-0.115 0 -0.032" rpy="0 ${pi/2} 0" />
     </joint>
- <joint name="quad_to_short_distance_lidar" type="fixed">
+    <joint name="quad_to_short_distance_lidar" type="fixed">
         <parent link="quad" />
         <child link="short_distance_lidar" />

Commit message: Update 1.5 urdf

File: robots/drone_1.5.urdf.xacro (robot description, xacro)
@@ -16,20 +16,20 @@
         <parent link="quad" />
         <child link="center_of_lift" />
-        <origin xyz="0 0 0.065" />
+        <origin xyz="0 0 0.055" />
     </joint>
     <joint name="quad_to_tfmini" type="fixed">
         <parent link="quad" />
         <child link="tfmini" />
-        <origin xyz="-0.115 0 -0.032" rpy="0 ${pi/2} 0" />
+        <origin xyz="-0.015 0.0925 -0.055" rpy="0 ${pi/2} 0" />
     </joint>
     <joint name="quad_to_short_distance_lidar" type="fixed">
         <parent link="quad" />
         <child link="short_distance_lidar" />
-        <origin xyz="0.08 -0.032 -0.035" rpy="0 ${pi/2} 0" />
+        <origin xyz="0.07 0.0925 -0.040" rpy="0 ${pi/2} 0" />
     </joint>
     <joint name="quad_to_base_footprint" type="fixed">
         <parent link="quad" />
         <child link="base_footprint" />
-        <origin xyz="0 0 -0.07" />
+        <origin xyz="0 0 -0.08" />
     </joint>
     <xacro:property name="foot_dist" value="0.1415" />

Commit message: Add PMW3901 optical frame for v1.5

File: robots/drone_1.5.urdf.xacro (robot description, xacro)
@@ -10,7 +10,5 @@
     <link name="foot3" />
     <link name="foot4" />
-    <!--
-    <link name="bottom_camera_link" />
-    -->
+    <link name="pmw3901_optical_flow" />
     <joint name="quad_to_center_of_lift" type="fixed">
         <parent link="quad" />
@@ -45,10 +43,8 @@
     <xacro:foot name="foot3" reflect_x="-1" reflect_y="-1" />
     <xacro:foot name="foot4" reflect_x="1" reflect_y="-1" />
-    <!--
     <joint name="quad_to_bottom_camera_link" type="fixed">
         <parent link="quad" />
-        <child link="bottom_camera_link" />
+        <child link="pmw3901_optical_flow" />
         <origin xyz="0 0 0" rpy="0 ${pi/2} 0" />
     </joint>
-    -->
 </robot>

Commit message: Add PMW3901 optical frame

File: robots/drone_1.5.urdf.xacro (robot description, xacro)
@@ -11,4 +11,5 @@
     <link name="foot4" />
     <link name="pmw3901_optical_flow" />
+    <link name="pmw3901_optical_flow_optical" />
     <joint name="quad_to_center_of_lift" type="fixed">
         <parent link="quad" />
@@ -48,3 +49,8 @@
         <origin xyz="0 0 0" rpy="0 ${pi/2} 0" />
     </joint>
+    <joint name="bottom_camera_link_to_optical" type="fixed">
+        <parent link="pmw3901_optical_flow" />
+        <child link="pmw3901_optical_flow_optical" />
+        <origin xyz="0 0 0" rpy="-${pi/2} 0 -${pi/2}" />
+    </joint>
 </robot>
