Commit message: Update launch files and urdf for 1.9

File: robots/drone_1.9.urdf.xacro (robot description, xacro)
@@ -20,17 +20,17 @@
         <parent link="quad" />
         <child link="tfmini" />
-        <origin xyz="-0.015 0.0925 -0.055" rpy="0 ${pi/2} 0" />
+        <origin xyz="0.14 -0.14 -0.05" rpy="0 ${pi/2} 0" />
     </joint>
     <joint name="quad_to_short_distance_lidar" type="fixed">
         <parent link="quad" />
         <child link="short_distance_lidar" />
-        <origin xyz="0.07 0.0925 -0.040" rpy="0 ${pi/2} 0" />
+        <origin xyz="-0.12 -0.12 -0.04" rpy="0 ${pi/2} 0" />
     </joint>
     <joint name="quad_to_base_footprint" type="fixed">
         <parent link="quad" />
         <child link="base_footprint" />
-        <origin xyz="0 0 -0.08" />
+        <origin xyz="0 0 -0.13" />
     </joint>
-    <xacro:property name="foot_dist" value="0.1415" />
+    <xacro:property name="foot_dist" value="0.155" />
     <xacro:macro name="foot" params="name reflect_x reflect_y">
         <joint name="base_footprint_to_${name}" type="fixed">
@@ -47,5 +47,5 @@
         <parent link="quad" />
         <child link="pmw3901_optical_flow" />
-        <origin xyz="0 0 0" rpy="0 ${pi/2} 0" />
+        <origin xyz="-0.14 -0.14 -0.04" rpy="0 ${-3*pi/4} 0" />
     </joint>
     <joint name="bottom_camera_link_to_optical" type="fixed">

Commit message: Fix typo and fix urdf transforms

File: robots/drone_1.9.urdf.xacro (robot description, xacro)
@@ -25,5 +25,5 @@
         <parent link="quad" />
         <child link="short_distance_lidar" />
-        <origin xyz="-0.12 -0.12 -0.04" rpy="0 ${pi/2} 0" />
+        <origin xyz="-0.12 0.12 -0.04" rpy="0 ${pi/2} 0" />
     </joint>
     <joint name="quad_to_base_footprint" type="fixed">
@@ -47,5 +47,5 @@
         <parent link="quad" />
         <child link="pmw3901_optical_flow" />
-        <origin xyz="-0.14 -0.14 -0.04" rpy="0 ${-3*pi/4} 0" />
+        <origin xyz="-0.14 -0.14 -0.04" rpy="0 ${pi/2} ${-3*pi/4}" />
     </joint>
     <joint name="bottom_camera_link_to_optical" type="fixed">

Commit message: Add r200 to v1.9

File: robots/drone_1.9.urdf.xacro (robot description, xacro)
@@ -46,4 +46,9 @@
     <joint name="quad_to_bottom_camera_link" type="fixed">
         <parent link="quad" />
+        <child link="bottom_camera_link" />
+        <origin xyz="-0.1 0 -0.04" rpy="0 ${pi/2} ${pi}" />
+    </joint>
+    <joint name="quad_to_bottom_camera_link" type="fixed">
+        <parent link="quad" />
         <child link="pmw3901_optical_flow" />
         <origin xyz="-0.14 -0.14 -0.04" rpy="0 ${pi/2} ${-3*pi/4}" />

Commit message: Fix mistakes in v1-9 camera files

File: robots/drone_1.9.urdf.xacro (robot description, xacro)
@@ -10,4 +10,5 @@
     <link name="foot3" />
     <link name="foot4" />
+    <link name="bottom_camera_link" />
     <link name="pmw3901_optical_flow" />
     <link name="pmw3901_optical_flow_optical" />
@@ -49,5 +50,5 @@
         <origin xyz="-0.1 0 -0.04" rpy="0 ${pi/2} ${pi}" />
     </joint>
-    <joint name="quad_to_bottom_camera_link" type="fixed">
+    <joint name="quad_to_pmw3901_optical_flow" type="fixed">
         <parent link="quad" />
         <child link="pmw3901_optical_flow" />
