Commit message: updated urdf for 2.0

File: robots/drone_2.0.urdf.xacro (robot description, xacro)
@@ -3,5 +3,5 @@
     <link name="quad" />
     <link name="center_of_lift" />
-    <link name="tfmini" />
+    <link name="lidarlite" />
     <link name="short_distance_lidar" />
     <link name="base_footprint" />
@@ -11,20 +11,18 @@
     <link name="foot4" />
     <link name="bottom_camera_link" />
-    <link name="pmw3901_optical_flow" />
-    <link name="pmw3901_optical_flow_optical" />
     <joint name="quad_to_center_of_lift" type="fixed">
         <parent link="quad" />
         <child link="center_of_lift" />
-        <origin xyz="0 0 0.055" />
+        <origin xyz="0 0 0.06" />
     </joint>
-    <joint name="quad_to_tfmini" type="fixed">
+    <joint name="quad_to_lidarlite" type="fixed">
         <parent link="quad" />
-        <child link="tfmini" />
-        <origin xyz="0.14 -0.14 -0.05" rpy="0 ${pi/2} 0" />
+        <child link="lidarlite" />
+        <origin xyz="-0.163 0.163 -0.05" rpy="0 ${pi/2} 0" />
     </joint>
     <joint name="quad_to_short_distance_lidar" type="fixed">
         <parent link="quad" />
         <child link="short_distance_lidar" />
-        <origin xyz="-0.12 0.12 -0.04" rpy="0 ${pi/2} 0" />
+        <origin xyz="0.304 0.304 -0.03" rpy="0 ${pi/2} 0" />
     </joint>
     <joint name="quad_to_base_footprint" type="fixed">
@@ -48,15 +46,5 @@
         <parent link="quad" />
         <child link="bottom_camera_link" />
-        <origin xyz="-0.1 0 -0.04" rpy="0 ${pi/2} ${pi}" />
-    </joint>
-    <joint name="quad_to_pmw3901_optical_flow" type="fixed">
-        <parent link="quad" />
-        <child link="pmw3901_optical_flow" />
-        <origin xyz="-0.14 -0.14 -0.04" rpy="0 ${pi/2} ${-3*pi/4}" />
-    </joint>
-    <joint name="bottom_camera_link_to_optical" type="fixed">
-        <parent link="pmw3901_optical_flow" />
-        <child link="pmw3901_optical_flow_optical" />
-        <origin xyz="0 0 0" rpy="-${pi/2} 0 -${pi/2}" />
+        <origin xyz="0 0 -0.065" rpy="0 ${pi/2} ${pi}" />
     </joint>
 </robot>

Commit message: 2.0 configuration files

File: robots/drone_2.0.urdf.xacro (robot description, xacro)
@@ -19,17 +19,17 @@
         <parent link="quad" />
         <child link="lidarlite" />
-        <origin xyz="-0.163 0.163 -0.05" rpy="0 ${pi/2} 0" />
+        <origin xyz="-0.163 0.163 0.02" rpy="0 ${pi/2} 0" />
     </joint>
     <joint name="quad_to_short_distance_lidar" type="fixed">
         <parent link="quad" />
         <child link="short_distance_lidar" />
-        <origin xyz="0.304 0.304 -0.03" rpy="0 ${pi/2} 0" />
+        <origin xyz="0.304 0.304 -0.043" rpy="0 ${pi/2} 0" />
     </joint>
     <joint name="quad_to_base_footprint" type="fixed">
         <parent link="quad" />
         <child link="base_footprint" />
-        <origin xyz="0 0 -0.13" />
+        <origin xyz="0 0 -0.10" />
     </joint>
-    <xacro:property name="foot_dist" value="0.155" />
+    <xacro:property name="foot_dist" value="0.233" />
     <xacro:macro name="foot" params="name reflect_x reflect_y">
         <joint name="base_footprint_to_${name}" type="fixed">
@@ -46,5 +46,5 @@
         <parent link="quad" />
         <child link="bottom_camera_link" />
-        <origin xyz="0 0 -0.065" rpy="0 ${pi/2} ${pi}" />
+        <origin xyz="0 0 -0.065" rpy="0 ${pi/2} 0" />
     </joint>
 </robot>

Commit message: added new tf for lidaaaaaar littteoo

File: robots/drone_2.0.urdf.xacro (robot description, xacro)
@@ -24,5 +24,5 @@
         <parent link="quad" />
         <child link="short_distance_lidar" />
-        <origin xyz="0.304 0.304 -0.043" rpy="0 ${pi/2} 0" />
+        <origin xyz="0.25 0.33-0.043" rpy="0 ${pi/2} 0" />
     </joint>
     <joint name="quad_to_base_footprint" type="fixed">

Commit message: Update 2.0's transforms

File: robots/drone_2.0.urdf.xacro (robot description, xacro)
@@ -24,10 +24,10 @@
         <parent link="quad" />
         <child link="short_distance_lidar" />
-        <origin xyz="0.25 0.33-0.043" rpy="0 ${pi/2} 0" />
+        <origin xyz="0.25 0.33 -0.043" rpy="0 ${pi/2} 0" />
     </joint>
     <joint name="quad_to_base_footprint" type="fixed">
         <parent link="quad" />
         <child link="base_footprint" />
-        <origin xyz="0 0 -0.10" />
+        <origin xyz="0 0 -0.215" />
     </joint>
     <xacro:property name="foot_dist" value="0.233" />
@@ -46,5 +46,5 @@
         <parent link="quad" />
         <child link="bottom_camera_link" />
-        <origin xyz="0 0 -0.065" rpy="0 ${pi/2} 0" />
+        <origin xyz="0 -0.0508 -0.065" rpy="0 ${pi/2} 0" />
     </joint>
 </robot>

Commit message: Update camera launch files

File: robots/drone_2.0.urdf.xacro (robot description, xacro)
@@ -11,4 +11,5 @@
     <link name="foot4" />
     <link name="bottom_camera_link" />
+    <link name="bottom_camera_rgb_optical_frame" />
     <joint name="quad_to_center_of_lift" type="fixed">
         <parent link="quad" />
@@ -46,5 +47,11 @@
         <parent link="quad" />
         <child link="bottom_camera_link" />
-        <origin xyz="0 -0.0508 -0.065" rpy="0 ${pi/2} 0" />
+        <origin xyz="0 0.07 -0.09" rpy="0 ${pi/2} -${pi/2}" />
+    </joint>
+    <joint name="bottom_camera_link_to_bottom_camera_rgb_optical_frame"
+        type="fixed">
+        <parent link="bottom_camera_link" />
+        <child link="bottom_camera_rgb_optical_frame" />
+        <origin rpy="-${pi/2} 0 -${pi/2}" />
     </joint>
 </robot>

Commit message: forward camera transform

File: robots/drone_2.0.urdf.xacro (robot description, xacro)
@@ -55,3 +55,13 @@
         <origin rpy="-${pi/2} 0 -${pi/2}" />
     </joint>
+    <joint name="quad_to_forward_camera_link" type="fixed">
+        <parent link="quad" />
+        <child link="forward_camera_link" />
+        <origin xyz="0.1 0 -0.04" rpy="0 0 0" />
+    </joint>
+    <joint name="forward_camera_link_to_optical" type="fixed">
+        <parent link="forward_camera_link" />
+        <child link="forward_camera_optical" />
+        <origin xyz="0 0 0" rpy="${-pi/2} 0 0" />
+    </joint>
 </robot>

Commit message: Add forward realsense to 2.0 base hardware

File: robots/drone_2.0.urdf.xacro (robot description, xacro)
@@ -63,5 +63,5 @@
         <parent link="forward_camera_link" />
         <child link="forward_camera_optical" />
-        <origin xyz="0 0 0" rpy="${-pi/2} 0 0" />
+        <origin xyz="0.2 -0.02 0" rpy="${-pi/2} 0 0" />
     </joint>
 </robot>

Commit message: Fix urdf 2.0

File: robots/drone_2.0.urdf.xacro (robot description, xacro)
@@ -12,4 +12,6 @@
     <link name="bottom_camera_link" />
     <link name="bottom_camera_rgb_optical_frame" />
+    <link name="forward_camera_link" />
+    <link name="forward_camera_optical" />
     <joint name="quad_to_center_of_lift" type="fixed">
         <parent link="quad" />

Commit message: Fix forward camera transform position, needs to be renamed

File: robots/drone_2.0.urdf.xacro (robot description, xacro)
@@ -13,5 +13,4 @@
     <link name="bottom_camera_rgb_optical_frame" />
     <link name="forward_camera_link" />
-    <link name="forward_camera_optical" />
     <joint name="quad_to_center_of_lift" type="fixed">
         <parent link="quad" />
@@ -60,10 +59,5 @@
         <parent link="quad" />
         <child link="forward_camera_link" />
-        <origin xyz="0.1 0 -0.04" rpy="0 0 0" />
-    </joint>
-    <joint name="forward_camera_link_to_optical" type="fixed">
-        <parent link="forward_camera_link" />
-        <child link="forward_camera_optical" />
-        <origin xyz="0.2 -0.02 0" rpy="${-pi/2} 0 0" />
+        <origin xyz="0.15 -0.02 -0.04" rpy="0 0 0" />
     </joint>
 </robot>

Commit message: Added side camera transforms

File: robots/drone_2.0.urdf.xacro (robot description, xacro)
@@ -12,5 +12,8 @@
     <link name="bottom_camera_link" />
     <link name="bottom_camera_rgb_optical_frame" />
-    <link name="forward_camera_link" />
+    <link name="front_camera_link" />
+    <link name="left_camera_link" />
+    <link name="right_camera_link" />
+    <link name="back_camera_link" />
     <joint name="quad_to_center_of_lift" type="fixed">
         <parent link="quad" />
@@ -56,8 +59,18 @@
         <origin rpy="-${pi/2} 0 -${pi/2}" />
     </joint>
-    <joint name="quad_to_forward_camera_link" type="fixed">
-        <parent link="quad" />
-        <child link="forward_camera_link" />
-        <origin xyz="0.15 -0.02 -0.04" rpy="0 0 0" />
-    </joint>
+    <xacro:property name="camera_z" value="-0.04" />
+    <xacro:property name="camera_horiz_offset" value="0.15" />
+    <xacro:macro name="side_camera" params="name pitch yaw">
+        <joint name="quad_to_${name}_camera_link" type="fixed">
+            <parent link="quad" />
+            <child link="${name}_camera_link" />
+            <origin
+                xyz="${camera_horiz_offset*cos(yaw)} ${camera_horiz_offset*sin(yaw)} ${camera_z}"
+                rpy="0 ${pitch} ${yaw}" />
+        </joint>
+    </xacro:macro>
+    <xacro:side_camera name="front" pitch="${20*pi/180}" yaw="${0*pi/2}" />
+    <xacro:side_camera name="left"  pitch="${35*pi/180}" yaw="${1*pi/2}" />
+    <xacro:side_camera name="back"  pitch="${20*pi/180}" yaw="${2*pi/2}" />
+    <xacro:side_camera name="right" pitch="${35*pi/180}" yaw="${3*pi/2}" />
 </robot>

Commit message: Updated side camera locations

File: robots/drone_2.0.urdf.xacro (robot description, xacro)
@@ -59,6 +59,6 @@
         <origin rpy="-${pi/2} 0 -${pi/2}" />
     </joint>
-    <xacro:property name="camera_z" value="-0.04" />
-    <xacro:property name="camera_horiz_offset" value="0.15" />
+    <xacro:property name="camera_z" value="-0.13" />
+    <xacro:property name="camera_horiz_offset" value="0.20" />
     <xacro:macro name="side_camera" params="name pitch yaw">
         <joint name="quad_to_${name}_camera_link" type="fixed">

Commit message: Update cameras and positions

File: robots/drone_2.0.urdf.xacro (robot description, xacro)
@@ -12,4 +12,5 @@
     <link name="bottom_camera_link" />
     <link name="bottom_camera_rgb_optical_frame" />
+    <link name="bottom_camera_r200_link" />
     <link name="front_camera_link" />
     <link name="left_camera_link" />
@@ -59,4 +60,9 @@
         <origin rpy="-${pi/2} 0 -${pi/2}" />
     </joint>
+    <joint name="quad_to_bottom_camera_r200_link" type="fixed">
+        <parent link="quad" />
+        <child link="bottom_camera_r200_link" />
+        <origin xyz="0 -0.05 -0.065" rpy="0 ${pi/2} ${0.1}" />
+    </joint>
     <xacro:property name="camera_z" value="-0.13" />
     <xacro:property name="camera_horiz_offset" value="0.20" />
@@ -71,6 +77,6 @@
     </xacro:macro>
     <xacro:side_camera name="front" pitch="${13*pi/180}" yaw="${0*pi/2}" />
-    <xacro:side_camera name="left"  pitch="${35*pi/180}" yaw="${1*pi/2}" />
+    <xacro:side_camera name="left"  pitch="${18.5*pi/180}" yaw="${1*pi/2}" />
     <xacro:side_camera name="back"  pitch="${15*pi/180}" yaw="${2*pi/2}" />
-    <xacro:side_camera name="right" pitch="${30*pi/180}" yaw="${3*pi/2}" />
+    <xacro:side_camera name="right" pitch="${13*pi/180}" yaw="${3*pi/2}" />
 </robot>

Commit message: on jetson

File: robots/drone_2.0.urdf.xacro (robot description, xacro)
@@ -59,5 +59,5 @@
         <parent link="quad" />
         <child link="forward_camera_link" />
-        <origin xyz="0.15 -0.02 -0.04" rpy="0 0 0" />
+        <origin xyz="-0.02 -0.15 -0.04" rpy="0 0 -${pi/2}" />
     </joint>
 </robot>
